File: modulinSchematic/modulinSchematic.kicad_sch (KiCad schematic)
At the start: 15 parts, among them U3 TL074, U4 TL074, U5 LM393

Commit message: Add power schematic
Parts:
- removed R5, R6, R7: R_US, Resistor_THT:R_Axial_DIN0207_L6.3mm_D2.5mm_P10.16mm_Horizontal, symbol Device:R_US
- removed RV4: 100k, Potentiometer_THT:Potentiometer_Bourns_3266Y_Vertical, symbol Device:R_Potentiometer_Trim_US
- removed U5: LM393, Package_DIP:DIP-8_W7.62mm, symbol Comparator:LM393
Connections:
- net at RV5.2: now also U4.2 (-)
- net at U4.3 (+): now also RV1.2, U3.3 (+)
- net GATE: now reaches U4.1
- net GATE: no longer U4.2 (-)
- net ADSR: no longer names the net of U4.6 (-)
- net ADSR: no longer U4.7
Other:
- sheet ADSR renamed ADSR_VCA
- sheet ADSR_VCA ports: added GATE_IN; removed none
- sheet VCA ports: added CV_IN; removed CV
- sheet VCF ports: added CV_IN; removed CV
- note removed: "Gate Generator"
- moved on the sheet: RV1, RV5, U3A, U4A, U4B, U4C, U4D
