File: modulinPowerSupply/modulinPowerSupply.kicad_sch (KiCad schematic)
At the start: 26 parts, among them J1 Barrel_Jack_Switch, J2 Screw_Terminal_01x04, U1 LM7812_TO220, U2 LM7912_TO220, U5 LM7805_TO220

Commit message: Write out envelope circuit and make PCB, edit PSU
Parts:
- removed C13, C14, C15: 4700uF, Capacitor_THT:CP_Radial_D16.0mm_P7.50mm, symbol Device:C_US
- removed C16, C17: 1uF, Capacitor_THT:CP_Radial_D4.0mm_P2.00mm, symbol Device:C_US
- removed D5, D6: 1N4001, Diode_THT:D_DO-41_SOD81_P10.16mm_Horizontal, symbol Diode:1N4001
- removed J1: Barrel_Jack_Switch, Connector_BarrelJack:BarrelJack_Horizontal, symbol Connector:Barrel_Jack_Switch
- removed J2: Screw_Terminal_01x04, TerminalBlock:TerminalBlock_Xinya_XY308-2.54-4P_1x04_P2.54mm_Horizontal, symbol Connector:Screw_Terminal_01x04
- removed U5: LM7805_TO220, Package_TO_SOT_THT:TO-220-3_Vertical, symbol Regulator_Linear:LM7805_TO220
- added J1: Screw_Terminal_01x02, User:TerminalBlock_1x2_CNC, symbol Connector:Screw_Terminal_01x02
- added J2: Screw_Terminal_01x03, User:TerminalBlock_1x3_CNC, symbol Connector:Screw_Terminal_01x03
- C1, C2, C3, C4, C5, C6: footprint Capacitor_THT:CP_Radial_D16.0mm_P7.50mm -> User:C_Radial_Polarized_P7.50mm_CNC
- C10, C7, C8, C9: footprint Capacitor_THT:CP_Radial_D4.0mm_P2.00mm -> User:C_Rect_P5.00mm_CNC
- D1, D2, D3, D4: footprint Diode_THT:D_DO-41_SOD81_P10.16mm_Horizontal -> User:D_P10.16mm_CNC
- U1, U2: footprint Package_TO_SOT_THT:TO-220-3_Vertical -> User:TO-220_CNC
Connections:
- net +12V: now also J2.3 (Pin_3)
- net -12V: now also J2.1 (Pin_1)
- net GND: now also J1.1 (Pin_1), J2.2 (Pin_2)
- net at D1.2 (A), D2.1 (K): now also J1.2 (Pin_2)
