File: modulinPowerSupply/modulinPowerSupply.kicad_pcb (KiCad board)
At the start: 2 copper layers, 25.4 x 177.8 mm, 23 parts, among them J1 Screw_Terminal_01x02, J2 Screw_Terminal_01x03, U1 LM7812_TO220, U2 LM7912_TO220

Commit message: Add STEP files
Other:
- board text added: "GND"
- board text added: "VCC"
- board text added: "VEE"
Changed lines of the file:
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@@
 		(tenting front back)
 		(pcbplotparams
-			(layerselection 0x00000000_00000000_55555555_57555554)
+			(layerselection 0x00000000_00000000_55555555_5755f5ff)
 			(plot_on_all_layers_selection 0x00000000_00000000_00000000_00000000)
 			(disableapertmacros no)
@@
 			(drillshape 0)
 			(scaleselection 1)
-			(outputdirectory "D:/Modulin/PSU/")
+			(outputdirectory "modulinPowerSupplyGerber/")
 		)
 	)
@@
 		(pad "1" thru_hole circle
 			(at 0 0)
-			(size 1.27 1.27)
+			(size 1.778 1.778)
 			(drill 1.27)
 			(layers "*.Cu" "*.Mask")
@@
 		(pad "2" thru_hole circle
 			(at 7.5 0)
-			(size 1.27 1.27)
+			(size 1.778 1.778)
 			(drill 1.27)
 			(layers "*.Cu" "*.Mask")
@@
 		(pad "1" thru_hole circle
 			(at 0 0)
-			(size 0.8128 0.8128)
+			(size 1.3208 1.3208)
 			(drill 0.8128)
 			(layers "*.Cu" "*.Mask")
@@
 		(pad "2" thru_hole circle
 			(at 5 0)
-			(size 0.8128 0.8128)
+			(size 1.3208 1.3208)
 			(drill 0.8128)
 			(layers "*.Cu" "*.Mask")
@@
 			)
 		)
-		(property "Datasheet" ""
+		(property "Datasheet" "~"
 			(at 0 0 90)
 			(layer "F.Fab")
@@
 		(pad "1" thru_hole circle
 			(at 0 0 270)
-			(size 1.397 1.397)
+			(size 1.905 1.905)
 			(drill 1.397)
 			(layers "*.Cu" "*.Mask")
@@
 		(pad "2" thru_hole circle
 			(at 5 0 270)
-			(size 1.397 1.397)
+			(size 1.905 1.905)
 			(drill 1.397)
 			(layers "*.Cu" "*.Mask")
@@
 		(pad "1" thru_hole circle
 			(at 0 0)
-			(size 0.8128 0.8128)
+			(size 1.3208 1.3208)
 			(drill 0.8128)
 			(layers "*.Cu" "*.Mask")
@@
 		(pad "2" thru_hole circle
 			(at 5 0)
-			(size 0.8128 0.8128)
+			(size 1.3208 1.3208)
 			(drill 0.8128)
 			(layers "*.Cu" "*.Mask")
@@
 		(pad "1" thru_hole circle
 			(at 0 0)
-			(size 1.27 1.27)
+			(size 1.778 1.778)
 			(drill 1.27)
 			(layers "*.Cu" "*.Mask")
@@
 		(pad "2" thru_hole circle
 			(at 7.5 0)
-			(size 1.27 1.27)
+			(size 1.778 1.778)
 			(drill 1.27)
 			(layers "*.Cu" "*.Mask")
@@
 		(pad "1" thru_hole circle
 			(at 0 0 180)
-			(size 0.8128 0.8128)
+			(size 1.3208 1.3208)
 			(drill 0.8128)
 			(layers "*.Cu" "*.Mask")
@@
 		(pad "2" thru_hole circle
 			(at 5 0 180)
-			(size 0.8128 0.8128)
+			(size 1.3208 1.3208)
 			(drill 0.8128)
 			(layers "*.Cu" "*.Mask")
@@
 		(pad "1" thru_hole circle
 			(at 0 0)
-			(size 1.27 1.27)
+			(size 1.778 1.778)
 			(drill 1.27)
 			(layers "*.Cu" "*.Mask")
@@
 		(pad "2" thru_hole circle
 			(at 7.5 0)
-			(size 1.27 1.27)
+			(size 1.778 1.778)
 			(drill 1.27)
 			(layers "*.Cu" "*.Mask")
@@
 		(pad "1" thru_hole circle
 			(at 0 0)
-			(size 0.8128 0.8128)
+			(size 1.3208 1.3208)
 			(drill 0.8128)
 			(layers "*.Cu" "*.Mask")
@@
 		(pad "2" thru_hole circle
 			(at 5 0)
-			(size 0.8128 0.8128)
+			(size 1.3208 1.3208)
 			(drill 0.8128)
 			(layers "*.Cu" "*.Mask")
@@
 			)
 		)
-		(property "Datasheet" ""
+		(property "Datasheet" "~"
 			(at 0 0 0)
 			(layer "F.Fab")
@@
 		(pad "1" thru_hole circle
 			(at 0 0 180)
-			(size 1.397 1.397)
+			(size 1.905 1.905)
 			(drill 1.397)
 			(layers "*.Cu" "*.Mask")
@@
 		(pad "2" thru_hole circle
 			(at 5 0 180)
-			(size 1.397 1.397)
+			(size 1.905 1.905)
 			(drill 1.397)
 			(layers "*.Cu" "*.Mask")
@@
 		(pad "3" thru_hole circle
 			(at 10 0 180)
-			(size 1.397 1.397)
+			(size 1.905 1.905)
 			(drill 1.397)
 			(layers "*.Cu" "*.Mask")
@@
 		(pad "1" thru_hole circle
 			(at 0 0)
-			(size 1.27 1.27)
+			(size 1.778 1.778)
 			(drill 1.27)
 			(layers "*.Cu" "*.Mask")
@@
 		(pad "2" thru_hole circle
 			(at 7.5 0)
-			(size 1.27 1.27)
+			(size 1.778 1.778)
 			(drill 1.27)
 			(layers "*.Cu" "*.Mask")
@@
 		(pad "1" thru_hole circle
 			(at 0 0)
-			(size 1.27 1.27)
+			(size 1.778 1.778)
 			(drill 1.27)
 			(layers "*.Cu" "*.Mask")
@@
 		(pad "2" thru_hole circle
 			(at 7.5 0)
-			(size 1.27 1.27)
+			(size 1.778 1.778)
 			(drill 1.27)
 			(layers "*.Cu" "*.Mask")
@@
 		(pad "1" thru_hole circle
 			(at 0 0)
-			(size 1.27 1.27)
+			(size 1.778 1.778)
 			(drill 1.27)
 			(layers "*.Cu" "*.Mask")
@@
 		(pad "2" thru_hole circle
 			(at 7.5 0)
-			(size 1.27 1.27)
+			(size 1.778 1.778)
 			(drill 1.27)
 			(layers "*.Cu" "*.Mask")
@@
 		(layer "Edge.Cuts")
 	)
+	(gr_text "VCC"
+		(at 33.02 183.642 0)
+		(layer "F.SilkS")
+		(effects
+			(font
+				(size 1 1)
+				(thickness 0.15)
+			)
+		)
+	)
+	(gr_text "VEE"
+		(at 43.18 183.642 0)
+		(layer "F.SilkS")
+		(effects
+			(font
+				(size 1 1)
+				(thickness 0.15)
+			)
+		)
+	)
+	(gr_text "GND"
+		(at 38.1 183.642 0)
+		(layer "F.SilkS")
+		(effects
+			(font
+				(size 1 1)
+				(thickness 0.15)
+			)
+		)
+	)
 	(segment
