File: modulinEnvelope/modulinEnvelope.kicad_sch (KiCad schematic)
At the start: 48 parts, among them J1 Conn_01x03_Socket, J2 Conn_01x03_Socket, Q1 BC548, Q2 BC548, Q3 BC548, Q4 BC548, Q5 BC548, Q6 BC548, Q7 2N7000, U1 TL074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

Commit message: Add VCF ciruit and edit for JLCPCB
Parts:
- removed J1, J2: Conn_01x03_Socket, User:TerminalBlock_1x3_CNC, symbol Connector:Conn_01x03_Socket
- added J1: Screw_Terminal_01x06, User:TerminalBlock_1x6_CNC, symbol Connector:Screw_Terminal_01x06
- U2: footprint User:DIP8_CNC -> User:DIP-8_CNC
Connections:
- net GATE: now also J1.6 (Pin_6)
- net GND: now also J1.2 (Pin_2)
- net VCC: now also J1.3 (Pin_3)
- net VEE: now also J1.1 (Pin_1)
- net ENV_VCA renamed OUT
- net OUT: now also J1.4 (Pin_4)
- net VCF_ENV renamed IN
- net IN: now also J1.5 (Pin_5)
Changed lines of the file:
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@@
 	(rectangle
 		(start 185.42 120.65)
-		(end 226.06 147.32)
+		(end 226.06 161.29)
 		(stroke
 			(width 0)
@@
 		)
 	)
-	(global_label "VCF_ENV"
+	(global_label "IN"
 		(shape input)
-		(at 212.09 135.89 0)
+		(at 193.04 135.89 0)
 		(fields_autoplaced yes)
 		(effects
@@
 		)
 		(property "Intersheetrefs" "${INTERSHEET_REFS}"
-			(at 223.0581 135.89 0)
+			(at 197.9605 135.89 0)
 			(effects
 				(font
@@
 		)
 	)
-	(global_label "ENV_VCA"
+	(global_label "OUT"
 		(shape input)
 		(at 140.97 138.43 0)
@@
 		)
 		(property "Intersheetrefs" "${INTERSHEET_REFS}"
-			(at 151.9381 138.43 0)
+			(at 147.5838 138.43 0)
 			(effects
 				(font
@@
 		)
 	)
-	(global_label "ENV_VCA"
+	(global_label "OUT"
 		(shape input)
-		(at 212.09 133.35 0)
+		(at 193.04 138.43 0)
 		(fields_autoplaced yes)
 		(effects
@@
 		)
 		(property "Intersheetrefs" "${INTERSHEET_REFS}"
-			(at 223.0581 133.35 0)
+			(at 199.6538 138.43 0)
 			(effects
 				(font
@@
 	(global_label "GATE"
 		(shape input)
-		(at 212.09 138.43 0)
+		(at 193.04 133.35 0)
 		(fields_autoplaced yes)
 		(effects
@@
 		)
 		(property "Intersheetrefs" "${INTERSHEET_REFS}"
-			(at 219.5504 138.43 0)
+			(at 200.5004 133.35 0)
 			(effects
 				(font
@@
 		)
 	)
-	(global_label "VCF_ENV"
+	(global_label "IN"
 		(shape input)
 		(at 66.04 138.43 180)
@@
 		)
 		(property "Intersheetrefs" "${INTERSHEET_REFS}"
-			(at 55.0719 138.43 0)
+			(at 61.1195 138.43 0)
 			(effects
 				(font
@@
 	)
 	(symbol
-		(lib_id "Connector:Conn_01x03_Socket")
-		(at 207.01 135.89 180)
-		(unit 1)
-		(exclude_from_sim no)
-		(in_bom yes)
-		(on_board yes)
-		(dnp no)
-		(property "Reference" "J2"
-			(at 207.645 128.27 0)
-			(effects
-				(font
-					(size 1.27 1.27)
-				)
-			)
-		)
-		(property "Value" "Conn_01x03_Socket"
-			(at 207.645 130.81 90)
-			(effects
-				(font
-					(size 1.27 1.27)
-				)
-				(hide yes)
-			)
-		)
-		(property "Footprint" "User:TerminalBlock_1x3_CNC"
-			(at 207.01 135.89 0)
-			(effects
-				(font
-					(size 1.27 1.27)
-				)
-				(hide yes)
-			)
-		)
-		(property "Datasheet" "~"
-			(at 207.01 135.89 0)
-			(effects
-				(font
-					(size 1.27 1.27)
-				)
-				(hide yes)
-			)
-		)
-		(property "Description" "Generic connector, single row, 01x03, script generated"
-			(at 207.01 135.89 0)
-			(effects
-				(font
-					(size 1.27 1.27)
-				)
-				(hide yes)
-			)
-		)
-		(pin "2"
-		)
-		(pin "1"
-		)
-		(pin "3"
-		)
-		(instances
-			(project "modulinEnvelope"
-				(path "/efb82606-78cb-466a-8666-7fc27cb05238"
-					(reference "J2")
-					(unit 1)
-				)
-			)
-		)
-	)
-	(symbol
 		(lib_id "Device:R")
 		(at 55.88 44.45 180)
@@
 	)
 	(symbol
-		(lib_id "Connector:Conn_01x03_Socket")
-		(at 191.77 135.89 180)
-		(unit 1)
-		(exclude_from_sim no)
-		(in_bom yes)
-		(on_board yes)
-		(dnp no)
-		(property "Reference" "J1"
-			(at 192.405 128.27 0)
-			(effects
-				(font
-					(size 1.27 1.27)
-				)
-			)
-		)
-		(property "Value" "Conn_01x03_Socket"
-			(at 192.405 130.81 90)
-			(effects
-				(font
-					(size 1.27 1.27)
-				)
-				(hide yes)
-			)
-		)
-		(property "Footprint" "User:TerminalBlock_1x3_CNC"
-			(at 191.77 135.89 0)
-			(effects
-				(font
-					(size 1.27 1.27)
-				)
-				(hide yes)
-			)
-		)
-		(property "Datasheet" "~"
-			(at 191.77 135.89 0)
-			(effects
-				(font
-					(size 1.27 1.27)
-				)
-				(hide yes)
-			)
-		)
-		(property "Description" "Generic connector, single row, 01x03, script generated"
-			(at 191.77 135.89 0)
-			(effects
-				(font
-					(size 1.27 1.27)
-				)
-				(hide yes)
-			)
-		)
-		(pin "2"
-		)
-		(pin "1"
-		)
-		(pin "3"
-		)
-		(instances
-			(project ""
-				(path "/efb82606-78cb-466a-8666-7fc27cb05238"
-					(reference "J1")
-					(unit 1)
-				)
-			)
-		)
-	)
-	(symbol
 		(lib_id "power:GND")
 		(at 101.6 55.88 0)
@@
 	(symbol
 		(lib_id "power:VEE")
-		(at 196.85 138.43 180)
+		(at 193.04 146.05 270)
 		(unit 1)
 		(exclude_from_sim no)
@@
 		(fields_autoplaced yes)
 		(property "Reference" "#PWR03"
-			(at 196.85 134.62 0)
+			(at 189.23 146.05 0)
 			(effects
 				(font
@@
 		)
 		(property "Value" "VEE"
-			(at 196.85 143.51 0)
+			(at 196.85 146.0499 90)
 			(effects
 				(font
 					(size 1.27 1.27)
 				)
+				(justify left)
 			)
 		)
 		(property "Footprint" ""
-			(at 196.85 138.43 0)
+			(at 193.04 146.05 0)
 			(effects
 				(font
@@
 		)
 		(property "Datasheet" ""
-			(at 196.85 138.43 0)
+			(at 193.04 146.05 0)
 			(effects
 				(font
@@
 		)
 		(property "Description" "Power symbol creates a global label with name \"VEE\""
-			(at 196.85 138.43 0)
+			(at 193.04 146.05 0)
 			(effects
 				(font
@@
 	(symbol
 		(lib_id "power:GND")
-		(at 196.85 135.89 90)
+		(at 193.04 143.51 90)
 		(unit 1)
 		(exclude_from_sim no)
@@
 		(fields_autoplaced yes)
 		(property "Reference" "#PWR01"
-			(at 203.2 135.89 0)
+			(at 199.39 143.51 0)
 			(effects
 				(font
@@
 		)
 		(property "Value" "GND"
-			(at 200.66 135.8899 90)
+			(at 196.85 143.5099 90)
 			(effects
 				(font
@@
 		)
 		(property "Footprint" ""
-			(at 196.85 135.89 0)
+			(at 193.04 143.51 0)
 			(effects
 				(font
@@
 		)
 		(property "Datasheet" ""
-			(at 196.85 135.89 0)
+			(at 193.04 143.51 0)
 			(effects
 				(font
@@
 		)
 		(property "Description" "Power symbol creates a global label with name \"GND\" , ground"
-			(at 196.85 135.89 0)
+			(at 193.04 143.51 0)
 			(effects
 				(font
@@
 	)
 	(symbol
+		(lib_id "Connector:Screw_Terminal_01x06")
+		(at 187.96 140.97 180)
+		(unit 1)
+		(exclude_from_sim no)
+		(in_bom yes)
+		(on_board yes)
+		(dnp no)
+		(fields_autoplaced yes)
+		(property "Reference" "J1"
+			(at 187.96 127 0)
+			(effects
+				(font
+					(size 1.27 1.27)
+				)
+			)
+		)
+		(property "Value" "Screw_Terminal_01x06"
+			(at 187.96 129.54 0)
+			(effects
+				(font
+					(size 1.27 1.27)
+				)
+			)
+		)
+		(property "Footprint" "User:TerminalBlock_1x6_CNC"
+			(at 187.96 140.97 0)
+			(effects
+				(font
+					(size 1.27 1.27)
+				)
+				(hide yes)
+			)
+		)
+		(property "Datasheet" "~"
+			(at 187.96 140.97 0)
+			(effects
+				(font
+					(size 1.27 1.27)
+				)
+				(hide yes)
+			)
+		)
+		(property "Description" "Generic screw terminal, single row, 01x06, script generated (kicad-library-utils/schlib/autogen/connector/)"
+			(at 187.96 140.97 0)
+			(effects
+				(font
+					(size 1.27 1.27)
+				)
+				(hide yes)
+			)
+		)
+		(pin "5"
+		)
+		(pin "2"
+		)
+		(pin "1"
+		)
+		(pin "6"
+		)
+		(pin "3"
+		)
+		(pin "4"
+		)
+		(instances
+			(project ""
+				(path "/efb82606-78cb-466a-8666-7fc27cb05238"
+					(reference "J1")
+					(unit 1)
+				)
+			)
+		)
+	)
+	(symbol
 		(lib_id "Diode:1N4148WT")
 		(at 208.28 72.39 0)
@@
 			)
 		)
-		(property "Footprint" "User:DIP8_CNC"
+		(property "Footprint" "User:DIP-8_CNC"
 			(at 140.97 58.42 0)
 			(effects
@@
 	(symbol
 		(lib_id "power:VCC")
-		(at 196.85 133.35 0)
+		(at 193.04 140.97 270)
 		(unit 1)
 		(exclude_from_sim no)
@@
 		(fields_autoplaced yes)
 		(property "Reference" "#PWR02"
-			(at 196.85 137.16 0)
+			(at 189.23 140.97 0)
 			(effects
 				(font
@@
 		)
 		(property "Value" "VCC"
-			(at 196.85 128.27 0)
+			(at 196.85 140.9699 90)
 			(effects
 				(font
 					(size 1.27 1.27)
 				)
+				(justify left)
 			)
 		)
 		(property "Footprint" ""
-			(at 196.85 133.35 0)
+			(at 193.04 140.97 0)
 			(effects
 				(font
@@
 		)
 		(property "Datasheet" ""
-			(at 196.85 133.35 0)
+			(at 193.04 140.97 0)
 			(effects
 				(font
@@
 		)
 		(property "Description" "Power symbol creates a global label with name \"VCC\""
-			(at 196.85 133.35 0)
+			(at 193.04 140.97 0)
 			(effects
 				(font

Commit message: Add STEP files
Connections:
- net at Q7.3 (D): now also RV5.1; no longer RV5.3
- net at R21.2: now also RV5.3; no longer RV5.1
Changed lines of the file:
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@@
 		(lib_id "Device:R_Potentiometer")
 		(at 163.83 73.66 0)
+		(mirror x)
 		(unit 1)
 		(exclude_from_sim no)
@@
 		(on_board yes)
 		(dnp no)
-		(fields_autoplaced yes)
 		(property "Reference" "RV5"
-			(at 161.29 72.3899 0)
+			(at 161.29 74.9301 0)
 			(effects
 				(font
@@
 		)
 		(property "Value" "B100k"
-			(at 161.29 74.9299 0)
+			(at 161.29 72.3901 0)
 			(effects
 				(font
