File: modulinEnvelope/modulinEnvelope.kicad_sch (KiCad schematic)
At the start: 47 parts, among them J1 Screw_Terminal_01x06, Q1 BC548, Q2 BC548, Q3 BC548, Q4 BC548, Q5 BC548, Q6 BC548, Q7 2N7000, U1 TL074, U2 NA555P

Commit message: Finish up CAD
Parts:
- R3, R4: value 1k 1% -> 10k 1%
Changed lines of the file:
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@@
 			)
 		)
-		(property "Value" "1k 1%"
+		(property "Value" "10k 1%"
 			(at 85.09 130.81 0)
 			(effects
@@
 			)
 		)
-		(property "Value" "1k 1%"
+		(property "Value" "10k 1%"
 			(at 104.14 130.81 0)
 			(effects
