File: modulinLFO/modulinLFO.kicad_pcb (KiCad board)
At the start: 2 copper layers, 88.9 x 177.8 mm, 118 parts, among them J1 Screw_Terminal_01x05, Q1 BC548, Q2 BC548, Q3 2N7000, Q4 BC548, Q5 BC548, Q6 BC548, Q7 BC548, Q8 BC548, SW1 SW_SPDT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

Commit message: Add STEP files
Parts:
- SW1: footprint User:SW_Slide_SPST_H6.00mm_CNC -> User:SW_Slide_SPDT_H6.00mm_CNC
- U7: footprint User:DIP8_CNC -> User:DIP-8_CNC
Connections:
- C1 pad 2: Net-(Q2-C) -> Net-(Q1-C)
- C2 pad 2: Net-(Q1-C) -> Net-(Q2-C)
- Q3 pad 1: Net-(Q1-C) -> Net-(Q2-C)
- R7 pad 2: Net-(Q2-C) -> Net-(Q1-C)
- RV1 pad 1: VCC -> VEE
- RV1 pad 3: VEE -> VCC
- RV16 pad 1: EXP -> GND
- RV16 pad 3: GND -> EXP
- RV2 pad 1: VCC -> VEE
- RV2 pad 3: VEE -> VCC
- RV3 pad 1: EXP -> GND
- RV3 pad 3: GND -> EXP
- U1 pad 2: Net-(Q2-C) -> Net-(Q1-C)
- U3 pad 6: Net-(Q1-C) -> Net-(Q2-C)
Routing:
- net VCC: track 548.9 -> 518.3 mm
- net VEE: track 376.0 -> 402.6 mm
- net GND: track 640.0 -> 658.1 mm
- net EXP: track 194.6 -> 211.0 mm
- net Net-(Q2-C): track 24.1 -> 35.0 mm
- net Net-(Q1-C): track 32.3 -> 31.2 mm, vias 0 -> 1
Other:
- board text added: "EXP"
- board text added: "Expression"
- board text added: "GND"
- board text added: "LFO"
- board text added: "Low Frequency Oscillator"
- board text added: "PWM"
- board text added: "Saw"
- board text added: "Sine"
- board text added: "Tri"
- board text added: "VCC"
- board text added: "VEE"
