File: modulinLFO/modulinLFO.kicad_pcb (KiCad board)
At the start: 2 copper layers, 88.9 x 177.8 mm, 118 parts, among them J1 Screw_Terminal_01x05, Q1 BC548, Q2 BC548, Q3 2N7000, Q4 BC548, Q5 BC548, Q6 BC548, Q7 BC548, Q8 BC548, SW1 SW_SPDT, SW2 SW_1x4, U1 TL074, U2 LM7805, U3 TL074, U4 TL074, U5 TL072, U6 TL072, U7 TL072, U8 TL072

Commit message: Finish up CAD
Parts:
- removed the R20 at (79.5, 95.2)
Routing:
- net Net-(U5B--): track 18.5 -> 2.54 mm
Changed lines of the file:
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@@
 		)
 	)
-	(footprint "User:R_5.08mm_CNC"
-		(layer "F.Cu")
-		(at 79.502 95.25 -90)
-		(descr "Resistor, Axial_DIN0204 series, Axial, Vertical, pin pitch=5.08mm, 0.167W, length*diameter=3.6*1.6mm^2, http://cdn-reichelt.de/documents/datenblatt/B400/1_4W%23YAG.pdf")
-		(tags "Resistor Axial_DIN0204 series Axial Vertical pin pitch 5.08mm 0.167W length 3.6mm diameter 1.6mm")
-		(property "Reference" "R20"
-			(at 2.54 -1.92 90)
-			(layer "F.SilkS")
-			(hide yes)
-			(effects
-				(font
-					(size 1 1)
-					(thickness 0.15)
-				)
-			)
-		)
-		(property "Value" "100k 1%"
-			(at 2.54 1.92 90)
-			(layer "F.Fab")
-			(effects
-				(font
-					(size 1 1)
-					(thickness 0.15)
-				)
-			)
-		)
-		(property "Datasheet" "~"
-			(at 0 0 270)
-			(unlocked yes)
-			(layer "F.Fab")
-			(hide yes)
-			(effects
-				(font
-					(size 1.27 1.27)
-					(thickness 0.15)
-				)
-			)
-		)
-		(property "Description" "Resistor"
-			(at 0 0 270)
-			(unlocked yes)
-			(layer "F.Fab")
-			(hide yes)
-			(effects
-				(font
-					(size 1.27 1.27)
-					(thickness 0.15)
-				)
-			)
-		)
-		(property ki_fp_filters "R_*")
-		(sheetname "/")
-		(sheetfile "modulinVCO.kicad_sch")
-		(attr through_hole)
-		(fp_line
-			(start 0.762 1.016)
-			(end 4.318 1.016)
-			(stroke
-				(width 0.1)
-				(type default)
-			)
-			(layer "F.SilkS")
-		)
-		(fp_line
-			(start 0.762 -1.016)
-			(end 4.318 -1.016)
-			(stroke
-				(width 0.1)
-				(type default)
-			)
-			(layer "F.SilkS")
-		)
-		(fp_line
-			(start -1.27 1.27)
-			(end 6.35 1.27)
-			(stroke
-				(width 0.05)
-				(type solid)
-			)
-			(layer "F.CrtYd")
-		)
-		(fp_line
-			(start 6.35 1.27)
-			(end 6.35 -1.27)
-			(stroke
-				(width 0.05)
-				(type solid)
-			)
-			(layer "F.CrtYd")
-		)
-		(fp_line
-			(start -1.27 -1.27)
-			(end -1.27 1.27)
-			(stroke
-				(width 0.05)
-				(type solid)
-			)
-			(layer "F.CrtYd")
-		)
-		(fp_line
-			(start 6.35 -1.27)
-			(end -1.27 -1.27)
-			(stroke
-				(width 0.05)
-				(type solid)
-			)
-			(layer "F.CrtYd")
-		)
-		(fp_line
-			(start 0 0)
-			(end 5.08 0)
-			(stroke
-				(width 0.1)
-				(type solid)
-			)
-			(layer "F.Fab")
-		)
-		(fp_circle
-			(center 0 0)
-			(end 0.8 0)
-			(stroke
-				(width 0.1)
-				(type solid)
-			)
-			(fill no)
-			(layer "F.Fab")
-		)
-		(fp_text user "${REFERENCE}"
-			(at 2.5 0 90)
-			(layer "F.SilkS")
-			(effects
-				(font
-					(size 1 1)
-					(thickness 0.15)
-				)
-			)
-		)
-		(fp_text user "${REFERENCE}"
-			(at 2.54 -1.92 90)
-			(layer "F.Fab")
-			(effects
-				(font
-					(size 1 1)
-					(thickness 0.15)
-				)
-			)
-		)
-		(pad "1" thru_hole circle
-			(at 0 0 270)
-			(size 1.3208 1.3208)
-			(drill 0.8128)
-			(layers "*.Cu" "*.Mask")
-			(remove_unused_layers no)
-			(net 38 "Net-(U5B--)")
-			(pintype "passive")
-		)
-		(pad "1" smd circle
-			(at 0 0 270)
-			(size 1.7272 1.7272)
-			(layers "B.Cu" "B.Mask" "B.Paste")
-			(net 38 "Net-(U5B--)")
-			(pintype "passive")
-		)
-		(pad "2" thru_hole circle
-			(at 5.08 0 270)
-			(size 1.6764 1.6764)
-			(drill 0.8128)
-			(layers "*.Cu" "*.Mask")
-			(remove_unused_layers no)
-			(net 35 "Net-(U4D--)")
-			(pintype "passive")
-		)
-		(embedded_fonts no)
-		(model "${KICAD9_3DMODEL_DIR}/Resistor_THT.3dshapes/R_Axial_DIN0204_L3.6mm_D1.6mm_P5.08mm_Vertical.wrl"
-			(offset
-				(xyz 0 0 0)
-			)
-			(scale
-				(xyz 1 1 1)
-			)
-			(rotate
-				(xyz 0 0 0)
-			)
-		)
-	)
 	(footprint "User:DIP-14_CNC"
 		(layer "F.Cu")
@@
 	)
 	(segment
-		(start 67.615822 89.154)
-		(end 73.711822 95.25)
-		(width 0.508)
-		(layer "B.Cu")
-		(net 38)
-	)
-	(segment
-		(start 66.04 89.154)
-		(end 67.615822 89.154)
-		(width 0.508)
-		(layer "B.Cu")
-		(net 38)
-	)
-	(segment
 		(start 66.04 86.614)
 		(end 66.04 89.154)
 		(width 0.508)
 		(layer "B.Cu")
-		(net 38)
-	)
-	(segment
-		(start 73.711822 95.25)
-		(end 79.502 95.25)
-		(width 0.508)
-		(layer "B.Cu")
