File: modulinLFO/modulinLFO.kicad_sch (KiCad schematic)
At the start: 112 parts, among them J1 Screw_Terminal_01x05, Q1 BC548, Q2 BC548, Q3 2N7000, Q4 BC548, Q5 BC548, Q6 BC548, Q7 BC548, Q8 BC548, SW1 SW_SPDT, SW2 SW_1x4, U1 TL074, U2 LM7805, U3 TL074, U4 TL074, U5 TL072, U6 TL072, U7 TL072, U8 TL072

Commit message: Finish up CAD
Parts:
- R38: value 18k -> 22k
Changed lines of the file:
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@@
 			)
 		)
-		(property "Value" "18k"
+		(property "Value" "22k"
 			(at 285.75 182.8799 0)
 			(effects
