File: modulinVCF/modulinVCF.kicad_pcb (KiCad board)
At the start: 2 copper layers, 50.8 x 177.8 mm, 74 parts, among them J1 Screw_Terminal_01x07, Q1 BC548, Q10 BC548, Q11 BC548, Q12 BC548, Q2 BC548, Q3 BC548, Q4 BC548, Q5 BC548, Q6 BC548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

Commit message: Add STEP files
Parts:
- RV3: value A100k -> C100k
- moved R26 2.79 mm to (65.8, 54.6)
Connections:
- R26 pad 1: GND -> Net-(U4B-+)
- R26 pad 2: Net-(U4B-+) -> Net-(R22-Pad1)
Routing:
- net Net-(U4B-+): track 57.2 -> 59.9 mm, vias 0 -> 1
- net Net-(R22-Pad1): track 40.7 -> 41.2 mm, vias 1 -> 0
Other:
- board text added: "EXP"
- board text added: "GND"
- board text added: "IN"
- board text added: "NOTE"
- board text added: "OUT"
- board text added: "VCC"
- board text added: "VEE"
Changed lines of the file:
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@@
 			(outputformat 1)
 			(mirror no)
-			(drillshape 1)
+			(drillshape 0)
 			(scaleselection 1)
-			(outputdirectory "")
+			(outputdirectory "modulinVCFGerber/")
 		)
 	)
@@
 			(layer "F.SilkS")
 		)
-		(fp_poly
-			(pts
-				(xy 0 3.92) (xy 0.44 4.53) (xy -0.44 4.53)
-			)
-			(stroke
-				(width 0.12)
-				(type solid)
-			)
-			(fill yes)
-			(layer "F.SilkS")
-		)
 		(fp_line
 			(start 33 4.31)
@@
 	(footprint "User:R_10.16mm_CNC"
 		(layer "F.Cu")
-		(at 68.58 54.61 180)
+		(at 65.786 54.61 180)
 		(descr "Resistor, Axial_DIN0207 series, Axial, Horizontal, pin pitch=10.16mm, 0.25W = 1/4W, length*diameter=6.3*2.5mm^2, http://cdn-reichelt.de/documents/datenblatt/B400/1_4W%23YAG.pdf")
 		(tags "Resistor Axial_DIN0207 series Axial Horizontal pin pitch 10.16mm 0.25W = 1/4W length 6.3mm diameter 2.5mm")
@@
 			(layers "*.Cu" "*.Mask")
 			(remove_unused_layers no)
-			(net 2 "GND")
+			(net 41 "Net-(U4B-+)")
 			(pintype "passive")
 		)
@@
 			(layers "*.Cu" "*.Mask")
 			(remove_unused_layers no)
-			(net 41 "Net-(U4B-+)")
+			(net 40 "Net-(R22-Pad1)")
 			(pintype "passive")
 		)
@@
 			)
 		)
-		(property "Value" "A100k"
+		(property "Value" "C100k"
 			(at 0 -10 0)
 			(layer "B.Fab")
@@
 		(layer "Edge.Cuts")
 	)
+	(gr_text "VEE"
+		(at 35.814 185.928 0)
+		(layer "F.SilkS")
+		(effects
+			(font
+				(size 1 1)
+				(thickness 0.15)
+			)
+		)
+	)
+	(gr_text "IN"
+		(at 60.96 185.928 0)
+		(layer "F.SilkS")
+		(effects
+			(font
+				(size 1 1)
+				(thickness 0.15)
+			)
+		)
+	)
+	(gr_text "OUT"
+		(at 66.04 185.928 0)
+		(layer "F.SilkS")
+		(effects
+			(font
+				(size 1 1)
+				(thickness 0.15)
+			)
+		)
+	)
+	(gr_text "VCC"
+		(at 45.974 185.928 0)
+		(layer "F.SilkS")
+		(effects
+			(font
+				(size 1 1)
+				(thickness 0.15)
+			)
+		)
+	)
+	(gr_text "NOTE"
+		(at 51.054 185.928 0)
+		(layer "F.SilkS")
+		(effects
+			(font
+				(size 1 1)
+				(thickness 0.15)
+			)
+		)
+	)
+	(gr_text "GND"
+		(at 41.148 185.928 0)
+		(layer "F.SilkS")
+		(effects
+			(font
+				(size 1 1)
+				(thickness 0.15)
+			)
+		)
+	)
+	(gr_text "EXP"
+		(at 56.134 185.928 0)
+		(layer "F.SilkS")
+		(effects
+			(font
+				(size 1 1)
+				(thickness 0.15)
+			)
+		)
+	)
 	(gr_text "Voltage Controlled\nFilter"
 		(at 50.8 25.146 0)
@@
 	)
 	(segment
-		(start 48.514 73.66)
-		(end 67.564 54.61)
+		(start 31.282 97.79)
+		(end 33.782 97.79)
 		(width 0.508)
 		(layer "F.Cu")
@@
 	)
 	(segment
-		(start 31.282 97.79)
-		(end 33.782 97.79)
+		(start 33.02 144.78)
+		(end 31.282 144.78)
 		(width 0.508)
 		(layer "F.Cu")
@@
 	)
 	(segment
-		(start 33.02 144.78)
-		(end 31.282 144.78)
+		(start 68.58 54.61)
+		(end 68.58 51.1)
 		(width 0.508)
 		(layer "F.Cu")
@@
 	)
 	(segment
-		(start 68.58 51.1)
-		(end 68.58 54.61)
-		(width 0.508)
-		(layer "F.Cu")
-		(net 2)
-	)
-	(segment
 		(start 70.82 149.86)
 		(end 68.58 147.62)
@@
 	)
 	(segment
-		(start 67.564 54.61)
-		(end 68.58 54.61)
+		(start 31.282 144.78)
+		(end 28.742 147.32)
 		(width 0.508)
 		(layer "F.Cu")
@@
 	)
 	(segment
-		(start 31.282 144.78)
-		(end 28.742 147.32)
+		(start 35.052 171.918)
+		(end 32.766 169.632)
 		(width 0.508)
 		(layer "F.Cu")
@@
 	)
 	(segment
-		(start 28.702 73.66)
-		(end 48.514 73.66)
+		(start 49.53 73.66)
+		(end 68.58 54.61)
 		(width 0.508)
 		(layer "F.Cu")
@@
 	)
 	(segment
-		(start 35.052 171.918)
-		(end 32.766 169.632)
+		(start 28.702 73.66)
+		(end 49.53 73.66)
 		(width 0.508)
 		(layer "F.Cu")
@@
 	)
 	(segment
-		(start 55.903 53.617)
+		(start 55.626 53.894)
 		(end 58.42 51.1)
 		(width 0.508)
@@
 		(net 40)
 	)
-	(via
-		(at 55.903 53.617)
-		(size 1.7272)
-		(drill 0.8128)
-		(layers "F.Cu" "B.Cu")
-		(net 40)
-	)
 	(segment
-		(start 42.159 49.276)
-		(end 42.164 49.281)
+		(start 55.626 54.61)
+		(end 55.626 53.894)
 		(width 0.508)
-		(layer "B.Cu")
+		(layer "F.Cu")
 		(net 40)
 	)
 	(segment
-		(start 52.4246 57.0494)
-		(end 42.926 57.0494)
+		(start 42.159 49.276)
+		(end 42.164 49.281)
 		(width 0.508)
 		(layer "B.Cu")
@@
 	)
 	(segment
-		(start 55.857 53.617)
-		(end 52.4246 57.0494)
+		(start 55.626 54.61)
+		(end 53.1866 57.0494)
 		(width 0.508)
 		(layer "B.Cu")
@@
 	)
 	(segment
-		(start 55.903 53.617)
-		(end 55.857 53.617)
+		(start 53.1866 57.0494)
+		(end 42.926 57.0494)
 		(width 0.508)
 		(layer "B.Cu")
@@
 	)
 	(segment
-		(start 59.99 54.61)
-		(end 63.5 51.1)
+		(start 63.5 51.1)
+		(end 63.5 54.61)
 		(width 0.508)
 		(layer "F.Cu")
@@
 	)
 	(segment
-		(start 58.42 54.61)
-		(end 59.99 54.61)
+		(start 65.786 54.61)
+		(end 63.5 54.61)
 		(width 0.508)
 		(layer "F.Cu")
@@
 	)
 	(segment
-		(start 47.841812 100.33)
-		(end 56.642 91.529812)
+		(start 61.214 54.61)
+		(end 56.642 59.182)
 		(width 0.508)
-		(layer "B.Cu")
+		(layer "F.Cu")
 		(net 41)
 	)
 	(segment
-		(start 56.642 91.529812)
-		(end 56.642 56.388)
+		(start 63.5 54.61)
+		(end 61.214 54.61)
+		(width 0.508)
+		(layer "F.Cu")
+		(net 41)
+	)
+	(via
+		(at 56.642 59.182)
+		(size 1.7272)
+		(drill 0.8128)
+		(layers "F.Cu" "B.Cu")
+		(net 41)
+	)
+	(segment
+		(start 47.841812 100.33)
+		(end 56.642 91.529812)
 		(width 0.508)
 		(layer "B.Cu")
@@
 	)
 	(segment
-		(start 56.642 56.388)
-		(end 58.42 54.61)
+		(start 56.642 91.529812)
+		(end 56.642 59.182)
 		(width 0.508)
 		(layer "B.Cu")
