File: modulinVCF/modulinVCF.kicad_pcb (KiCad board)
At the start: 2 copper layers, 50.8 x 177.8 mm, 74 parts, among them J1 Screw_Terminal_01x07, Q1 BC548, Q10 BC548, Q11 BC548, Q12 BC548, Q2 BC548, Q3 BC548, Q4 BC548, Q5 BC548, Q6 BC548, Q7 BC548, Q8 BC548, Q9 BC548, U1 TL074, U2 LM7805, U3 TL074, U4 TL072

Commit message: Finish up CAD
Parts:
- moved C15 17.5 mm to (47.2, 89.2)
- moved C16 17.5 mm to (28.7, 100.3)
Connections:
- U4 pad 4: VCC -> VEE
- U4 pad 8: VEE -> VCC
Routing:
- net VEE: track 278.6 -> 267.6 mm
- net VCC: track 260.9 -> 269.0 mm
Changed lines of the file:
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@@
 	(footprint "User:C_Axial_P5.00mm_CNC"
 		(layer "F.Cu")
-		(at 33.742 100.33 180)
+		(at 47.244 89.154 180)
 		(descr "C, Rect series, Radial, pin pitch=5.00mm, length*width=7*2.5mm^2, Capacitor")
 		(tags "C Rect series Radial pin pitch 5.00mm length 7mm width 2.5mm Capacitor")
@@
 			(layers "*.Cu" "*.Mask")
 			(remove_unused_layers no)
-			(net 1 "VCC")
+			(net 3 "VEE")
 			(pinfunction "V-")
 			(pintype "power_in")
@@
 			(size 2.54 1.7272)
 			(layers "B.Cu" "B.Mask" "B.Paste")
-			(net 1 "VCC")
+			(net 3 "VEE")
 			(pinfunction "V-")
 			(pintype "power_in")
@@
 			(layers "*.Cu" "*.Mask")
 			(remove_unused_layers no)
-			(net 3 "VEE")
+			(net 1 "VCC")
 			(pinfunction "V+")
 			(pintype "power_in")
@@
 			(size 2.54 1.7272)
 			(layers "B.Cu" "B.Mask" "B.Paste")
-			(net 3 "VEE")
+			(net 1 "VCC")
 			(pinfunction "V+")
 			(pintype "power_in")
@@
 	(footprint "User:C_Axial_P5.00mm_CNC"
 		(layer "F.Cu")
-		(at 42.204 89.154)
+		(at 28.702 100.33)
 		(descr "C, Rect series, Radial, pin pitch=5.00mm, length*width=7*2.5mm^2, Capacitor")
 		(tags "C Rect series Radial pin pitch 5.00mm length 7mm width 2.5mm Capacitor")
@@
 	(segment
 		(start 30.734 75.692)
-		(end 49.784 75.692)
+		(end 47.244 75.692)
 		(width 0.508)
 		(layer "F.Cu")
@@
 		(net 1)
 	)
+	(segment
+		(start 47.244 75.692)
+		(end 49.784 75.692)
+		(width 0.508)
+		(layer "F.Cu")
+		(net 1)
+	)
+	(segment
+		(start 47.244 89.154)
+		(end 47.244 75.692)
+		(width 0.508)
+		(layer "F.Cu")
+		(net 1)
+	)
 	(via
 		(at 30.734 75.692)
@@
 	)
 	(segment
-		(start 33.742 100.33)
-		(end 30.734 100.33)
-		(width 0.508)
-		(layer "B.Cu")
-		(net 1)
-	)
-	(segment
 		(start 30.734 171.704)
 		(end 30.734 161.29)
@@
 	)
 	(segment
-		(start 33.742 100.33)
-		(end 39.624 100.33)
+		(start 47.244 89.154)
+		(end 47.244 92.71)
 		(width 0.508)
 		(layer "B.Cu")
@@
 	)
 	(segment
+		(start 42.204 89.154)
+		(end 28.702 89.154)
+		(width 0.508)
+		(layer "F.Cu")
+		(net 2)
+	)
+	(segment
 		(start 68.58 54.61)
 		(end 68.58 51.1)
@@
 	)
 	(segment
-		(start 42.204 89.154)
-		(end 28.702 89.154)
-		(width 0.508)
-		(layer "F.Cu")
-		(net 2)
-	)
-	(segment
 		(start 70.82 149.86)
 		(end 68.58 147.62)
@@
 	)
 	(segment
-		(start 54.148 187.452)
-		(end 68.58 173.02)
+		(start 31.162 102.87)
+		(end 26.67 102.87)
 		(width 0.508)
 		(layer "F.Cu")
@@
 	)
 	(segment
-		(start 48.046 62.524)
-		(end 51.348 59.222)
+		(start 54.148 187.452)
+		(end 68.58 173.02)
 		(width 0.508)
 		(layer "F.Cu")
@@
 	)
 	(segment
-		(start 47.204 89.154)
-		(end 45.172 87.122)
+		(start 48.046 62.524)
+		(end 51.348 59.222)
 		(width 0.508)
 		(layer "F.Cu")
@@
 	)
 	(segment
+		(start 33.702 100.33)
+		(end 31.162 102.87)
+		(width 0.508)
+		(layer "F.Cu")
+		(net 3)
+	)
+	(segment
 		(start 51.348 59.222)
 		(end 52.367603 58.202397)
@@
 	)
 	(segment
-		(start 45.172 87.122)
-		(end 26.67 87.122)
-		(width 0.508)
-		(layer "F.Cu")
-		(net 3)
-	)
-	(segment
 		(start 51.348 59.262)
 		(end 51.348 59.222)
@@
 	)
 	(via
-		(at 36.04 184.912)
+		(at 26.67 102.87)
 		(size 1.7272)
 		(drill 0.8128)
@@
 	)
 	(via
-		(at 26.67 87.122)
+		(at 36.04 184.912)
 		(size 1.7272)
 		(drill 0.8128)
@@
 	)
 	(segment
-		(start 26.67 156.718)
+		(start 26.67 102.87)
 		(end 26.67 87.122)
 		(width 0.508)
@@
 	)
 	(segment
-		(start 47.244 92.71)
-		(end 47.244 89.194)
-		(width 0.508)
-		(layer "B.Cu")
-		(net 3)
-	)
-	(segment
 		(start 26.67 173.228)
 		(end 26.67 156.718)
@@
 	)
 	(segment
-		(start 47.244 89.194)
-		(end 47.204 89.154)
+		(start 26.67 156.718)
+		(end 26.67 102.87)
 		(width 0.508)
 		(layer "B.Cu")
@@
 		(width 0.508)
 		(layer "B.Cu")
+		(net 3)
+	)
+	(segment
+		(start 33.702 100.33)
+		(end 39.624 100.33)
+		(width 0.508)
+		(layer "B.Cu")
