File: modulinVCF/modulinVCF.kicad_sch (KiCad schematic)
At the start: 69 parts, among them J1 Screw_Terminal_01x07, Q1 BC548, Q10 BC548, Q11 BC548, Q12 BC548, Q2 BC548, Q3 BC548, Q4 BC548, Q5 BC548, Q6 BC548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

Commit message: Add STEP files
Parts:
- RV3: value A100k -> C100k
Connections:
- net GND: no longer R26.1
- net at R22.1, R24.2, RV3.3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: now also R26.2
- net at RV3.2, U4.5 (+): now also R26.1; no longer R26.2
Other:
- moved on the sheet: R26
Changed lines of the file:
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@@
 	)
 	(junction
-		(at 81.28 78.74)
-		(diameter 0)
-		(color 0 0 0 0)
-	)
-	(junction
 		(at 59.69 114.3)
 		(diameter 0)
@@
 	)
 	(junction
+		(at 85.09 62.23)
+		(diameter 0)
+		(color 0 0 0 0)
+	)
+	(junction
 		(at 271.78 58.42)
 		(diameter 0)
@@
 	)
 	(junction
-		(at 78.74 69.85)
+		(at 167.64 144.78)
 		(diameter 0)
 		(color 0 0 0 0)
 	)
 	(junction
-		(at 167.64 144.78)
+		(at 78.74 69.85)
 		(diameter 0)
 		(color 0 0 0 0)
@@
 	(wire
 		(pts
-			(xy 78.74 69.85) (xy 81.28 69.85)
+			(xy 71.12 69.85) (xy 78.74 69.85)
 		)
 		(stroke
@@
 	(wire
 		(pts
-			(xy 81.28 80.01) (xy 81.28 78.74)
-		)
-		(stroke
-			(width 0)
-			(type default)
-		)
-	)
-	(wire
-		(pts
 			(xy 160.02 93.98) (xy 165.1 93.98)
 		)
@@
 	(wire
 		(pts
-			(xy 85.09 78.74) (xy 85.09 73.66)
-		)
-		(stroke
-			(width 0)
-			(type default)
-		)
-	)
-	(wire
-		(pts
 			(xy 132.08 63.5) (xy 146.05 63.5)
 		)
@@
 	(wire
 		(pts
-			(xy 85.09 45.72) (xy 85.09 66.04)
+			(xy 85.09 45.72) (xy 85.09 62.23)
 		)
 		(stroke
@@
 	(wire
 		(pts
-			(xy 78.74 77.47) (xy 78.74 78.74)
-		)
-		(stroke
-			(width 0)
-			(type default)
-		)
-	)
-	(wire
-		(pts
 			(xy 138.43 83.82) (xy 172.72 83.82)
 		)
@@
 	(wire
 		(pts
-			(xy 71.12 69.85) (xy 78.74 69.85)
+			(xy 78.74 69.85) (xy 81.28 69.85)
 		)
 		(stroke
@@
 	(wire
 		(pts
-			(xy 81.28 78.74) (xy 78.74 78.74)
+			(xy 218.44 149.86) (xy 227.33 149.86)
 		)
 		(stroke
@@
 	(wire
 		(pts
-			(xy 218.44 149.86) (xy 227.33 149.86)
+			(xy 261.62 43.18) (xy 271.78 43.18)
 		)
 		(stroke
@@
 	(wire
 		(pts
-			(xy 261.62 43.18) (xy 271.78 43.18)
+			(xy 100.33 35.56) (xy 100.33 43.18)
 		)
 		(stroke
@@
 	(wire
 		(pts
-			(xy 100.33 35.56) (xy 100.33 43.18)
+			(xy 119.38 147.32) (xy 119.38 133.35)
 		)
 		(stroke
@@
 	(wire
 		(pts
-			(xy 119.38 147.32) (xy 119.38 133.35)
+			(xy 124.46 147.32) (xy 119.38 147.32)
 		)
 		(stroke
@@
 	(wire
 		(pts
-			(xy 124.46 147.32) (xy 119.38 147.32)
+			(xy 128.27 43.18) (xy 113.03 43.18)
 		)
 		(stroke
@@
 	(wire
 		(pts
-			(xy 128.27 43.18) (xy 113.03 43.18)
+			(xy 78.74 62.23) (xy 85.09 62.23)
 		)
 		(stroke
@@
 	(wire
 		(pts
-			(xy 181.61 99.06) (xy 172.72 99.06)
+			(xy 85.09 62.23) (xy 85.09 66.04)
 		)
 		(stroke
@@
 	(wire
 		(pts
-			(xy 146.05 73.66) (xy 146.05 78.74)
+			(xy 181.61 99.06) (xy 172.72 99.06)
 		)
 		(stroke
@@
 	(wire
 		(pts
-			(xy 81.28 78.74) (xy 85.09 78.74)
+			(xy 146.05 73.66) (xy 146.05 78.74)
 		)
 		(stroke
@@
 			)
 		)
-		(property "Value" "A100k"
+		(property "Value" "C100k"
 			(at 87.63 68.5801 0)
 			(effects
@@
 	(symbol
 		(lib_id "Device:R")
-		(at 78.74 73.66 0)
+		(at 78.74 66.04 0)
 		(mirror x)
 		(unit 1)
@@
 		(fields_autoplaced yes)
 		(property "Reference" "R26"
-			(at 76.2 72.3899 0)
+			(at 76.2 64.7699 0)
 			(effects
 				(font
@@
 		)
 		(property "Value" "10k"
-			(at 76.2 74.9299 0)
+			(at 76.2 67.3099 0)
 			(effects
 				(font
@@
 		)
 		(property "Footprint" "User:R_10.16mm_CNC"
-			(at 76.962 73.66 90)
+			(at 76.962 66.04 90)
 			(effects
 				(font
@@
 		)
 		(property "Datasheet" "~"
-			(at 78.74 73.66 0)
+			(at 78.74 66.04 0)
 			(effects
 				(font
@@
 		)
 		(property "Description" "Resistor"
-			(at 78.74 73.66 0)
+			(at 78.74 66.04 0)
 			(effects
 				(font
@@
 	(symbol
 		(lib_id "power:GND")
-		(at 81.28 80.01 0)
+		(at 85.09 73.66 0)
 		(unit 1)
 		(exclude_from_sim no)
@@
 		(fields_autoplaced yes)
 		(property "Reference" "#PWR029"
-			(at 81.28 86.36 0)
+			(at 85.09 80.01 0)
 			(effects
 				(font
@@
 		)
 		(property "Value" "GND"
-			(at 81.28 85.09 0)
+			(at 85.09 78.74 0)
 			(effects
 				(font
@@
 		)
 		(property "Footprint" ""
-			(at 81.28 80.01 0)
+			(at 85.09 73.66 0)
 			(effects
 				(font
@@
 		)
 		(property "Datasheet" ""
-			(at 81.28 80.01 0)
+			(at 85.09 73.66 0)
 			(effects
 				(font
@@
 		)
 		(property "Description" "Power symbol creates a global label with name \"GND\" , ground"
-			(at 81.28 80.01 0)
+			(at 85.09 73.66 0)
 			(effects
 				(font
