File: modulinVCF/modulinVCF.kicad_sch (KiCad schematic)
At the start: 69 parts, among them J1 Screw_Terminal_01x07, Q1 BC548, Q10 BC548, Q11 BC548, Q12 BC548, Q2 BC548, Q3 BC548, Q4 BC548, Q5 BC548, Q6 BC548, Q7 BC548, Q8 BC548, Q9 BC548, U1 TL074, U2 LM7805, U3 TL074, U4 TL072

Commit message: Finish up CAD
Connections:
- net VCC: now also U4.8 (V+); no longer U4.4 (V-)
- net VEE: now also U4.4 (V-); no longer U4.8 (V+)
Other:
- moved on the sheet: U4C
Changed lines of the file:
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@@
 	(symbol
 		(lib_id "Amplifier_Operational:TL072")
-		(at 259.08 50.8 180)
+		(at 259.08 50.8 0)
+		(mirror y)
 		(unit 3)
 		(exclude_from_sim no)
@@
 		(on_board yes)
 		(dnp no)
-		(fields_autoplaced yes)
 		(property "Reference" "U4"
-			(at 262.89 49.5299 0)
+			(at 262.89 52.0701 0)
 			(effects
 				(font
@@
 		)
 		(property "Value" "TL072"
-			(at 262.89 52.0699 0)
+			(at 262.89 49.5301 0)
 			(effects
 				(font
