File: modulinVCA/modulinVCA.kicad_sch (KiCad schematic)
At the start: 44 parts, among them J1 Screw_Terminal_01x08, Q1 BC548, Q2 BC548, Q3 BC548, Q4 BC548, Q5 BC548, Q6 BC548, U1 TL074

Commit message: Finish up CAD
Parts:
- RV4: value B1M -> B500k
Changed lines of the file:
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@@
 			)
 		)
-		(property "Value" "B1M"
+		(property "Value" "B500k"
 			(at 132.08 59.6901 0)
 			(effects
